File: hardware/horse-brain.sch (KiCad schematic (older format))
At the start: 45 parts, among them P1 M200, P2 Power in, Q3 2N7000, Q4 2N7000, Q5 2N7000

Commit message: Add fuel cell load and monitoring
Parts:
- added P?: Fuel cell, symbol CONN_2
- added R?: 47k, symbol R
Connections:
- net GND: now also P?.2 (PM), R?.2
- net at ARDUINO1.25 (A6): now also P?.1 (P1), R?.1
